File: labathome_pcb/labathome_pcb.kicad_sch (KiCad schematic)
At the start: 46 parts, among them J15 CAN RS 485, J17 Micro_SD_Card_Det1, J2 I2C, J21 GPIO, J22 Volts, J5 USB_ESP32, J6 PROG ESP, Q6 IRLML6344, SW1 Reset, SW6 YELLOW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

Commit message: Lab@Home 15.3 PCB as ordered @ JLCPCB
Parts:
- J6: footprint Connector:Tag-Connect_TC2030-IDC-NL_2x03_P1.27mm_Vertical -> liebler_CONN:IDC_2x03_P1.27mm_Vertical
Changed lines of the file:
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@@
 			)
 		)
-		(property "Footprint" "Connector:Tag-Connect_TC2030-IDC-NL_2x03_P1.27mm_Vertical"
+		(property "Footprint" "liebler_CONN:IDC_2x03_P1.27mm_Vertical"
 			(at 205.74 87.63 0)
 			(effects
